File: mouse_robot/mouse_robot.kicad_pcb (KiCad board)
At the start: 2 copper layers, 101.6 x 53.3 mm, 13 parts, among them J1 Power, J2 PWM, J3 Analog, J4 PWM, J5 Analog, J6 Communication, J7 Digital

Commit message: primeira ideia pronta
Parts:
- added D1: LED, LED_THT:LED_D3.0mm, B.Cu at (138.3, 55.5)
- added D2: LED, LED_THT:LED_D3.0mm, B.Cu at (162.2, 55.5)
- added D3: LED, LED_THT:LED_D3.0mm, B.Cu at (132.3, 55.5)
- added D4: LED, LED_THT:LED_D3.0mm, B.Cu at (156.2, 55.5)
- added D5: LED, LED_THT:LED_D3.0mm, B.Cu at (126.3, 55.5)
- added D6: LED, LED_THT:LED_D3.0mm, B.Cu at (150.3, 55.5)
- added D7: LED, LED_THT:LED_D3.0mm, B.Cu at (120.3, 55.5)
- added D8: LED, LED_THT:LED_D3.0mm, B.Cu at (144.3, 55.5)
- added J8: MPU-9250, Connector_PinSocket_2.54mm:PinSocket_1x08_P2.54mm_Vertical, B.Cu at (129.2, 84.8)
- added SW1: SW_MEC_5G, Button_Switch_THT:SW_PUSH_6mm, B.Cu at (112.8, 61.9)
- added SW2: SW_MEC_5G, Button_Switch_THT:SW_PUSH_6mm, B.Cu at (112.8, 70.5)
- added SW3: SW_MEC_5G, Button_Switch_THT:SW_PUSH_6mm, B.Cu at (112.8, 79.0)
- added SW4: SW_MEC_5G, Button_Switch_THT:SW_PUSH_6mm, B.Cu at (112.8, 87.6)
- added U1: tb66, ponteH:MODULE_ROB-14450, B.Cu at (179.0, 73.3)
- added con1: MOTOR2, Connector_Molex:Molex_KK-254_AE-6410-02A_1x02_P2.54mm_Vertical, B.Cu at (173.7, 89.8)
- added con2: MOTOR1, Connector_Molex:Molex_KK-254_AE-6410-02A_1x02_P2.54mm_Vertical, B.Cu at (171.1, 56.8)
- added con3: ENC1, Connector_Molex:Molex_KK-254_AE-6410-04A_1x04_P2.54mm_Vertical, B.Cu at (180.0, 56.8)
- added con4: ENC2, Connector_Molex:Molex_KK-254_AE-6410-04A_1x04_P2.54mm_Vertical, B.Cu at (187.6, 89.8)
- added con5: Bateria, Connector_Molex:Molex_KK-254_AE-6410-02A_1x02_P2.54mm_Vertical, B.Cu at (162.2, 87.3)

Commit message: componentes ok
Parts:
- removed D8: LED, LED_THT:LED_D3.0mm
- removed the J8 at (129.2, 84.8)
- removed SW3, SW4: SW_MEC_5G, Button_Switch_THT:SW_PUSH_6mm
- added J1: GND, Connector_Molex:Molex_KK-254_AE-6410-04A_1x04_P2.54mm_Vertical, B.Cu at (180.0, 61.9)
- added J11: I2C, Connector_Molex:Molex_KK-254_AE-6410-02A_1x02_P2.54mm_Vertical, B.Cu at (187.7, 56.8)
- added J12: ADC, Connector_Molex:Molex_KK-254_AE-6410-04A_1x04_P2.54mm_Vertical, B.Cu at (180.0, 92.4)
- added J13: MPU-9250, Connector_Molex:Molex_KK-254_AE-6410-10A_1x10_P2.54mm_Vertical, B.Cu at (127.9, 90.7)
- added J14: Display LCD, Connector_Molex:Molex_KK-254_AE-6410-12A_1x12_P2.54mm_Vertical, B.Cu at (121.6, 97.5)
- added J15: GPIO, Connector_Molex:Molex_KK-254_AE-6410-12A_1x12_P2.54mm_Vertical, B.Cu at (187.6, 92.4)
- added J2: 5V, Connector_Molex:Molex_KK-254_AE-6410-04A_1x04_P2.54mm_Vertical, B.Cu at (180.0, 77.1)
- added J7: BATERIA, Connector_Molex:Molex_KK-254_AE-6410-04A_1x04_P2.54mm_Vertical, B.Cu at (172.4, 56.9)
- added MUX: Conn_01x08_Socket, Connector_Molex:Molex_KK-254_AE-6410-08A_1x08_P2.54mm_Vertical, B.Cu at (158.5, 56.9)
- added R1: 220, Resistor_SMD:R_1206_3216Metric, B.Cu at (161.1, 93.7)
- added R2: 10k, Resistor_SMD:R_1206_3216Metric, B.Cu at (127.7, 65.7)
- added R3: 220, Resistor_SMD:R_1206_3216Metric, B.Cu at (106.8, 60.6)
- added R4: 220, Resistor_SMD:R_1206_3216Metric, B.Cu at (110.2, 60.6)
- added R5: 220, Resistor_SMD:R_1206_3216Metric, B.Cu at (113.6, 60.6)
- added R6: 220, Resistor_SMD:R_1206_3216Metric, B.Cu at (117.0, 60.6)
- added R7: 220, Resistor_SMD:R_1206_3216Metric, B.Cu at (120.4, 60.6)
- added R8: 220, Resistor_SMD:R_1206_3216Metric, B.Cu at (123.7, 60.6)
- added RV1: Potenciometro, Potentiometer_THT:Potentiometer_Vishay_T73YP_Vertical, B.Cu at (112.6, 75.9)
- D1, D2, D3, D4, D5, D6, D7: footprint LED_THT:LED_D3.0mm -> LED_SMD:LED_1206_3216Metric
- SW1: value SW_MEC_5G -> SW_Push; footprint Button_Switch_THT:SW_PUSH_6mm -> Button_Switch_THT:SW_PUSH_6mm_H4.3mm
- SW2: value SW_MEC_5G -> Power; footprint Button_Switch_THT:SW_PUSH_6mm -> Button_Switch_THT:SW_E-Switch_EG1271_SPDT
- moved D2 55.4 mm to (106.8, 55.5), turned to -90 degrees
- moved con3 47.5 mm to (134.3, 69.5)
- moved con4 47.1 mm to (141.9, 78.7)
- moved SW2 46.9 mm to (156.0, 88.9), turned to 0 degrees
- moved D4 42.7 mm to (113.6, 55.5), turned to -90 degrees
- moved D1 42.0 mm to (155.9, 93.7), turned to 0 degrees
- moved D6 29.9 mm to (120.4, 55.5), turned to -90 degrees
- moved con2 27.3 mm to (147.0, 69.5)
- moved con1 26.6 mm to (149.5, 78.7)
- moved D3 22.1 mm to (110.2, 55.5), turned to -90 degrees
- moved SW1 18.2 mm to (129.6, 54.8), turned to -90 degrees
- moved U1 15.3 mm to (163.8, 72.1), turned to 0 degrees
- moved con5 10.2 mm to (172.4, 87.3), turned to 180 degrees
- moved D5 9.34 mm to (117.0, 55.5), turned to -90 degrees
- moved D7 3.43 mm to (123.7, 55.5), turned to -90 degrees
- renumbered J6 to J10, J1 to J3, J3 to J4, J7 to J6, J2 to J8, J4 to J9
Connections:
- D1 pad 1: unconnected-(D1-K-Pad1) -> +5V
- D1 pad 2: unconnected-(D1-A-Pad2) -> Net-(D1-A)
- D2 pad 1: unconnected-(D2-K-Pad1) -> led1
- D2 pad 2: unconnected-(D2-A-Pad2) -> Net-(D2-A)
- D3 pad 1: unconnected-(D3-K-Pad1) -> led2
- D3 pad 2: unconnected-(D3-A-Pad2) -> Net-(D3-A)
- D4 pad 1: unconnected-(D4-K-Pad1) -> led3
- D4 pad 2: unconnected-(D4-A-Pad2) -> Net-(D4-A)
- D5 pad 1: unconnected-(D5-K-Pad1) -> led4
- D5 pad 2: unconnected-(D5-A-Pad2) -> Net-(D5-A)
- D6 pad 1: unconnected-(D6-K-Pad1) -> led5
- D6 pad 2: unconnected-(D6-A-Pad2) -> Net-(D6-A)
- D7 pad 1: unconnected-(D7-K-Pad1) -> led6
- D7 pad 2: unconnected-(D7-A-Pad2) -> Net-(D7-A)
- SW1 pad 1: Net-(SW1-A-Pad1) -> +5V
- SW1 pad 2: Net-(SW1-A-Pad1) -> btn1
- SW2 pad 1: Net-(SW2-A-Pad1) -> VCC
- SW2 pad 2: Net-(SW2-A-Pad1) -> Net-(SW2A-B)
- U1 pad 1: BAT -> VCC
- con5 pad 1: unconnected-(con5-Pin_1-Pad1) -> GND
- con5 pad 2: unconnected-(con5-Pin_2-Pad2) -> Net-(SW2A-B)

Commit message: roteamento init
Parts:
- SW2: value Power -> SW_DPDT_x2
- moved con4 7.62 mm to (134.3, 78.6), turned to 0 degrees
- moved SW2 5.41 mm to (160.6, 86.0), turned to 180 degrees
- moved con1 2.54 mm to (147.0, 78.7), turned to 0 degrees
- turned R1 to 180 degrees
- renumbered MUX to MUX1
Connections:
- J10 pad 1: /TX3/14 -> C1
- J10 pad 2: /RX3/15 -> C2
- J10 pad 3: /TX2/16 -> C3
- J10 pad 5: /TX1/18 -> ENC21
- J10 pad 6: /RX1/19 -> ENC22
- J10 pad 7: /SDA/20 -> SDA
- J10 pad 8: /SCL/21 -> SCL
- J11 pad 2: SDL -> SCL
- J13 pad 1: FYSINC -> unconnected-(J13-Pin_1-Pad1)
- J13 pad 2: NCS -> unconnected-(J13-Pin_2-Pad2)
- J13 pad 3: INT -> unconnected-(J13-Pin_3-Pad3)
- J13 pad 4: AD0 -> GND
- J13 pad 5: EDL -> unconnected-(J13-Pin_5-Pad5)
- J13 pad 6: EDA -> unconnected-(J13-Pin_6-Pad6)
- J13 pad 8: SDL -> SCL
- J4 pad 8: /A7 -> S0
- J5 pad 1: /A8 -> AD0
- J5 pad 2: /A9 -> AD1
- J5 pad 3: /A10 -> AD2
- J5 pad 4: /A11 -> AD3
- J6 pad 11: /*44 -> GPIO9
- J6 pad 13: /42 -> GPIO8
- J6 pad 14: /43 -> D7
- J6 pad 15: /40 -> GPIO7
- J6 pad 16: /41 -> D6
- J6 pad 17: /38 -> GPIO6
- J6 pad 18: /39 -> D5
- J6 pad 19: /36 -> GPIO5
- J6 pad 20: /37 -> D4
- J6 pad 21: /34 -> GPIO4
- J6 pad 22: /35 -> E
- J6 pad 23: /32 -> GPIO3
- J6 pad 24: /33 -> RW
- J6 pad 25: /30 -> GPIO2
- J6 pad 26: /31 -> RS
- J6 pad 27: /28 -> GPIO1
- J6 pad 29: /26 -> GPIO0
- J6 pad 31: /24 -> AI1
- J6 pad 32: /25 -> Ai2
- J6 pad 33: /22 -> BI2
- J6 pad 34: /23 -> BI1
- J6 pad 7: /48 -> GPIO11
- J6 pad 9: /*46 -> GPIO10
- J8 pad 1: /SCL/21 -> SCL
- J8 pad 10: /*8 -> led5
- J8 pad 2: /SDA/20 -> SDA
- J8 pad 6: /*12 -> led1
- J8 pad 7: /*11 -> led2
- J8 pad 8: /*10 -> led3
- J8 pad 9: /*9 -> led4
- J9 pad 1: /*7 -> led6
- J9 pad 2: /*6 -> EN
- J9 pad 3: /*5 -> PWMA
- J9 pad 4: /*4 -> PWMB
- J9 pad 5: /*3 -> btn1
- J9 pad 6: /*2 -> ENC11
- J9 pad 7: /TX0/1 -> C0
- J9 pad 8: /RX0/0 -> ENC12
- SW2 pad 1: VCC -> unconnected-(SW2A-A-Pad1)
- SW2 pad 2: Net-(SW2A-B) -> VCC
- SW2 pad 3: VCC -> Net-(SW2A-C)
- SW2 pad 4: Net-(SW2A-B) -> unconnected-(SW2B-A-Pad4)
- SW2 pad 5: (no net) -> VCC
- SW2 pad 6: (no net) -> Net-(SW2A-C)
- con5 pad 2: Net-(SW2A-B) -> Net-(SW2A-C)
Routing:
- net SDA: track 0.00 -> 130.2 mm
- net RS: track 0.00 -> 90.0 mm
- net RW: track 0.00 -> 88.2 mm
- net E: track 0.00 -> 86.4 mm
- net D4: track 0.00 -> 83.2 mm
- net D5: track 0.00 -> 81.6 mm
- net D7: track 0.00 -> 81.2 mm
- net D6: track 0.00 -> 80.1 mm
- net SCL: track 0.00 -> 59.6 mm
- net ENC22: track 0.00 -> 57.2 mm
- net ENC21: track 0.00 -> 56.0 mm
- net S0: track 0.00 -> 44.8 mm, vias 0 -> 1
- net PWMA: track 0.00 -> 42.0 mm
- net Ai2: track 0.00 -> 38.1 mm
- net ENC12: track 0.00 -> 34.3 mm
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
Commit message: pronto
Parts:
- moved SW2 5.90 mm to (155.5, 89.0), turned to 0 degrees
- renumbered MUX1 to MUX
Routing:
- net +5V: track 0.00 -> 210.8 mm
- net SCL: track 59.6 -> 128.1 mm
- net VCC: track 0.00 -> 59.9 mm
- net Net-(SW2A-C): track 0.00 -> 13.2 mm
- net btn1: track 24.1 -> 33.7 mm
- net S0: track 44.8 -> 46.0 mm
- added copper zone on B.Cu, net GND
- added copper zone on F.Cu, net GND
