File: mouse_robot/mouse_robot.kicad_sch (KiCad schematic)
At the start: 7 parts, among them J1 Power, J2 PWM, J3 Analog, J4 PWM, J5 Analog, J6 Communication, J7 Digital

Commit message: primeira ideia pronta
Parts:
- added D1, D2, D3, D4, D5, D6, D7, D8: LED, LED_THT:LED_D3.0mm, symbol Device:LED
- added J8: MPU-9250, Connector_PinSocket_2.54mm:PinSocket_1x08_P2.54mm_Vertical, symbol Connector:Conn_01x08_Socket
- added SW1, SW2, SW3, SW4: SW_MEC_5G, Button_Switch_THT:SW_PUSH_6mm, symbol Switch:SW_MEC_5G
- added U1: tb66, ponteH:MODULE_ROB-14450, symbol ponteH:ROB-14450
- added con1: MOTOR2, Connector_Molex:Molex_KK-254_AE-6410-02A_1x02_P2.54mm_Vertical, symbol Connector:Conn_01x02_Socket
- added con2: MOTOR1, Connector_Molex:Molex_KK-254_AE-6410-02A_1x02_P2.54mm_Vertical, symbol Connector:Conn_01x02_Socket
- added con3: ENC1, Connector_Molex:Molex_KK-254_AE-6410-04A_1x04_P2.54mm_Vertical, symbol Connector:Conn_01x04_Pin
- added con4: ENC2, Connector_Molex:Molex_KK-254_AE-6410-04A_1x04_P2.54mm_Vertical, symbol Connector:Conn_01x04_Pin
- added con5: Bateria, Connector_Molex:Molex_KK-254_AE-6410-02A_1x02_P2.54mm_Vertical, symbol Connector:Conn_01x02_Socket
Connections:
- net +5V: now also U1.13 (STBY), U1.2 (VCC), con3.1 (Pin_1), con4.1 (Pin_1)
- net GND: now also U1.3 (GND), U1.8 (GND), U1.9 (GND), con3.4 (Pin_4), con4.4 (Pin_4)
- new net: SW1.1 (A), SW1.2 (A)
- new net: SW1.3 (B), SW1.4 (B)
- new net: SW3.1 (A), SW3.2 (A)
- new net: SW3.3 (B), SW3.4 (B)
- new net: U1.5 (A02), con1.1 (Pin_1)
- new net: U1.4 (A01), con1.2 (Pin_2)
- new net: SW2.1 (A), SW2.2 (A)
- new net: SW2.3 (B), SW2.4 (B)
- new net: SW4.1 (A), SW4.2 (A)
- new net: SW4.3 (B), SW4.4 (B)
- new net: U1.6 (B02), con2.2 (Pin_2)
- new net: U1.7 (B01), con2.1 (Pin_1)
- new net AI1: U1.14 (AI1)
- new net Ai2: U1.15 (AI2)
- new net BAT: U1.1 (VM)
- new net BI1: U1.12 (BI1)
- new net BI2: U1.11 (BI2)
- new net ENC11: con3.2 (Pin_2)
- new net ENC12: con3.3 (Pin_3)
- new net ENC21: con4.2 (Pin_2)
- new net ENC22: con4.3 (Pin_3)
- new net PWMA: U1.16 (PWMA)
- new net PWMB: U1.10 (PWMB)
Other:
- note added: "Arduino Mega"
- moved on the sheet: J1, J2, J3, J4, J5, J6, J7

Commit message: eletric scheme ok
Parts:
- removed J8: MPU-9250, Connector_PinSocket_2.54mm:PinSocket_1x08_P2.54mm_Vertical, symbol Connector:Conn_01x08_Socket
- added D9: LED, LED_SMD:LED_1206_3216Metric, symbol Device:LED
- added J10: MUX, symbol Connector:Conn_01x07_Socket
- added J11: Display LCD, symbol Connector:Conn_01x12_Socket
- added J12: 5V, symbol Connector:Conn_01x04_Socket
- added J13: BATERIA, symbol Connector:Conn_01x04_Socket
- added J14: GPIO, symbol Connector:Conn_01x12_Socket
- added J15: ADC, symbol Connector:Conn_01x04_Pin
- added J16: I2C, symbol Connector:Conn_01x02_Pin
- added J8: MPU-9250, symbol Connector:Conn_01x10_Socket
- added J9: GND, symbol Connector:Conn_01x04_Socket
- added R1, R13, R2, R3, R4, R5, R6, R7, R8: 220, Resistor_SMD:R_1206_3216Metric, symbol Device:R_US
- added R10, R11, R12, R9: 10k, Resistor_SMD:R_1206_3216Metric, symbol Device:R_US
- added RV1: Potenciometro, symbol Device:R_Potentiometer_Trim_US
- added SW5: Power, symbol Switch:SW_DPST_x2
- D1, D2, D3, D4, D5, D6, D7, D8: footprint LED_THT:LED_D3.0mm -> LED_SMD:LED_1206_3216Metric
Connections:
- net BAT is gone; now on net VCC: U1.1 (VM)
- net +5V: now also SW1.1 (A), SW1.2 (A), SW2.1 (A), SW2.2 (A), SW3.1 (A), SW3.2 (A), SW4.1 (A), SW4.2 (A), D9.1 (K), J10.7 (Pin_7), J11.3 (Pin_3), J11.4 (Pin_4), J12.1 (Pin_1), J12.2 (Pin_2), J12.3 (Pin_3), J12.4 (Pin_4), J8.10 (Pin_10), RV1.1
- net GND: now also con5.1 (Pin_1), J10.1 (Pin_1), J11.1 (Pin_1), J11.2 (Pin_2), J8.1 (Pin_1), J9.1 (Pin_1), J9.2 (Pin_2), J9.3 (Pin_3), J9.4 (Pin_4), R1.1, R10.1, R11.1, R12.1, R13.1, R2.1, R3.1, R4.1, R5.1, R6.1, R7.1, R8.1, R9.1, RV1.3
- net VCC: now also J13.1 (Pin_1), J13.2 (Pin_2), J13.3 (Pin_3), J13.4 (Pin_4), SW5.1 (A), SW5.3 (A)
- net led7: now reaches D7.1 (K)
- net at D7.2 (A): now also R7.2
- net btn1: now reaches SW1.3 (B), SW1.4 (B)
- net btn1: now also R9.2
- net led5: now reaches D5.1 (K)
- net at D5.2 (A): now also R5.2
- net btn3: now reaches SW3.3 (B), SW3.4 (B)
- net btn3: now also SW4.3 (B), SW4.4 (B), R11.2, R12.2
- net at con5.2 (Pin_2): now also SW5.2 (B), SW5.4 (B)
- net led4: now reaches D4.1 (K)
- net at D4.2 (A): now also R4.2
- net led8: now reaches D8.1 (K)
- net at D8.2 (A): now also R8.2
- net led1: now reaches D1.1 (K)
- net at D1.2 (A): now also R1.2
- net btn2: now reaches SW2.3 (B), SW2.4 (B)
- net btn2: now also R10.2
- net led6: now reaches D6.1 (K)
- net at D6.2 (A): now also R6.2
- net led3: now reaches D3.1 (K)
- net at D3.2 (A): now also R3.2
- net led2: now reaches D2.1 (K)
- net at D2.2 (A): now also R2.2
- new net: D9.2 (A), R13.2
- new net: J11.12 (Pin_12), RV1.2
- new net AD0: J15.1 (Pin_1), J8.5 (Pin_5)
- new net AD1: J15.2 (Pin_2)
- new net AD2: J15.3 (Pin_3)
- new net AD3: J15.4 (Pin_4)
- new net C0: J10.5 (Pin_5)
- new net C1: J10.4 (Pin_4)
- new net C2: J10.3 (Pin_3)
- new net C3: J10.2 (Pin_2)
- new net D4: J11.8 (Pin_8)
- new net D5: J11.7 (Pin_7)
- new net D6: J11.6 (Pin_6)
- new net D7: J11.5 (Pin_5)
- new net E: J11.9 (Pin_9)
- new net EDA: J8.7 (Pin_7)
- new net EDL: J8.6 (Pin_6)
- new net FYSINC: J8.2 (Pin_2)
- new net GPIO0: J14.12 (Pin_12)
- new net GPIO1: J14.11 (Pin_11)
- new net GPIO10: J14.2 (Pin_2)
- new net GPIO11: J14.1 (Pin_1)
- new net GPIO2: J14.10 (Pin_10)
- new net GPIO3: J14.9 (Pin_9)
- new net GPIO4: J14.8 (Pin_8)
- new net GPIO5: J14.7 (Pin_7)
- new net GPIO6: J14.6 (Pin_6)
- new net GPIO7: J14.5 (Pin_5)
- new net GPIO8: J14.4 (Pin_4)
- new net GPIO9: J14.3 (Pin_3)
- new net INT: J8.4 (Pin_4)
- new net NCS: J8.3 (Pin_3)
- new net RS: J11.11 (Pin_11)
- new net RW: J11.10 (Pin_10)
- new net S0: J10.6 (Pin_6)
- new net SDA: J16.1 (Pin_1), J8.9 (Pin_9)
- new net SDL: J16.2 (Pin_2), J8.8 (Pin_8)
Other:
- title: (none) -> MOUSE ROBOT
- moved on the sheet: J1, J2, J3, J4, J5, J6, J7, SW1

Commit message: componentes ok
Parts:
- removed D7, D8: LED, LED_SMD:LED_1206_3216Metric, symbol Device:LED
- removed J10: MUX, symbol Connector:Conn_01x07_Socket
- removed R10, R11, R12: 10k, Resistor_SMD:R_1206_3216Metric, symbol Device:R_US
- removed R7, R8: 220, Resistor_SMD:R_1206_3216Metric, symbol Device:R_US
- removed SW1, SW2, SW3, SW4: SW_MEC_5G, Button_Switch_THT:SW_PUSH_6mm, symbol Switch:SW_MEC_5G
- added MUX: Conn_01x08_Socket, Connector_Molex:Molex_KK-254_AE-6410-08A_1x08_P2.54mm_Vertical, symbol Connector:Conn_01x08_Socket
- added SW1: SW_Push, Button_Switch_THT:SW_PUSH_6mm_H4.3mm, symbol Switch:SW_Push
- J1: renamed from J9; footprint (none) -> Connector_Molex:Molex_KK-254_AE-6410-04A_1x04_P2.54mm_Vertical
- J11: renamed from J16; footprint (none) -> Connector_Molex:Molex_KK-254_AE-6410-02A_1x02_P2.54mm_Vertical
- J12: renamed from J15; footprint (none) -> Connector_Molex:Molex_KK-254_AE-6410-04A_1x04_P2.54mm_Vertical
- J13: renamed from J8; footprint (none) -> Connector_Molex:Molex_KK-254_AE-6410-10A_1x10_P2.54mm_Vertical
- J14: renamed from J11; footprint (none) -> Connector_Molex:Molex_KK-254_AE-6410-12A_1x12_P2.54mm_Vertical
- J15: renamed from J14; footprint (none) -> Connector_Molex:Molex_KK-254_AE-6410-12A_1x12_P2.54mm_Vertical
- J2: renamed from J12; footprint (none) -> Connector_Molex:Molex_KK-254_AE-6410-04A_1x04_P2.54mm_Vertical
- J7: renamed from J13; footprint (none) -> Connector_Molex:Molex_KK-254_AE-6410-04A_1x04_P2.54mm_Vertical
- RV1: footprint (none) -> Potentiometer_THT:Potentiometer_Vishay_T73YP_Vertical
- SW2: renamed from SW5; footprint (none) -> Button_Switch_THT:SW_E-Switch_EG1271_SPDT
- renumbered D9 to D1, D1 to D2, D2 to D3, D3 to D4, D4 to D5, D5 to D6, D6 to D7, J6 to J10, J1 to J3, J3 to J4, J7 to J6, J2 to J8, J4 to J9, R13 to R1, R9 to R2, R1 to R3, R2 to R4, R3 to R5, R4 to R6, R5 to R7, R6 to R8
Connections:
- net +5V: now also MUX.7 (Pin_7), SW1.1
- net AD0: now also J13.4 (Pin_4); no longer J13.5 (Pin_5)
- net C0: now also MUX.5 (Pin_5)
- net C1: now also MUX.4 (Pin_4)
- net C2: now also MUX.3 (Pin_3)
- net C3: now also MUX.2 (Pin_2)
- net EDA: now also J13.6 (Pin_6); no longer J13.7 (Pin_7)
- net EDL: now also J13.5 (Pin_5); no longer J13.6 (Pin_6)
- net FYSINC: now also J13.1 (Pin_1); no longer J13.2 (Pin_2)
- net GND: now also J13.9 (Pin_9), MUX.8 (Pin_8); no longer J13.1 (Pin_1)
- net INT: now also J13.3 (Pin_3); no longer J13.4 (Pin_4)
- net NCS: now also J13.2 (Pin_2); no longer J13.3 (Pin_3)
- net S0: now also MUX.1 (Pin_1)
- net SDA: now also J13.7 (Pin_7); no longer J13.9 (Pin_9)
- net btn1: now also SW1.2
- new net EN: MUX.6 (Pin_6)

Commit message: roteamento init
Parts:
- removed SW2: Power, Button_Switch_THT:SW_E-Switch_EG1271_SPDT, symbol Switch:SW_DPST_x2
- added SW2: SW_DPDT_x2, symbol Switch:SW_DPDT_x2
- renumbered MUX to MUX1
Connections:
- net *10 is gone; now on net led3: J8.8 (Pin_8)
- net *11 is gone; now on net led2: J8.7 (Pin_7)
- net *12 is gone; now on net led1: J8.6 (Pin_6)
- net *2 is gone; now on net ENC11: J9.6 (Pin_6)
- net *3 is gone; now on net btn1: J9.5 (Pin_5)
- net *4 is gone; now on net PWMB: J9.4 (Pin_4)
- net *44 is gone; now on net GPIO9: J6.11 (Pin_11)
- net *46 is gone; now on net GPIO10: J6.9 (Pin_9)
- net *5 is gone; now on net PWMA: J9.3 (Pin_3)
- net *6 is gone; now on net EN: J9.2 (Pin_2)
- net *7 is gone; now on net led6: J9.1 (Pin_1)
- net *8 is gone; now on net led5: J8.10 (Pin_10)
- net *9 is gone; now on net led4: J8.9 (Pin_9)
- net 22 is gone; now on net BI2: J6.33 (Pin_33)
- net 23 is gone; now on net BI1: J6.34 (Pin_34)
- net 24 is gone; now on net AI1: J6.31 (Pin_31)
- net 25 is gone; now on net Ai2: J6.32 (Pin_32)
- net 26 is gone; now on net GPIO0: J6.29 (Pin_29)
- net 28 is gone; now on net GPIO1: J6.27 (Pin_27)
- net 30 is gone; now on net GPIO2: J6.25 (Pin_25)
- net 31 is gone; now on net RS: J6.26 (Pin_26)
- net 32 is gone; now on net GPIO3: J6.23 (Pin_23)
- net 33 is gone; now on net RW: J6.24 (Pin_24)
- net 34 is gone; now on net GPIO4: J6.21 (Pin_21)
- net 35 is gone; now on net E: J6.22 (Pin_22)
- net 36 is gone; now on net GPIO5: J6.19 (Pin_19)
- net 37 is gone; now on net D4: J6.20 (Pin_20)
- net 38 is gone; now on net GPIO6: J6.17 (Pin_17)
- net 39 is gone; now on net D5: J6.18 (Pin_18)
- net 40 is gone; now on net GPIO7: J6.15 (Pin_15)
- net 41 is gone; now on net D6: J6.16 (Pin_16)
- net 42 is gone; now on net GPIO8: J6.13 (Pin_13)
- net 43 is gone; now on net D7: J6.14 (Pin_14)
- net 48 is gone; now on net GPIO11: J6.7 (Pin_7)
- net A10 is gone; now on net AD2: J5.3 (Pin_3)
- net A11 is gone; now on net AD3: J5.4 (Pin_4)
- net A7 is gone; now on net S0: J4.8 (Pin_8)
- net A8 is gone; now on net AD0: J5.1 (Pin_1)
- net A9 is gone; now on net AD1: J5.2 (Pin_2)
- net RX0/0 is gone; now on net ENC12: J9.8 (Pin_8)
- net RX1/19 is gone; now on net ENC22: J10.6 (Pin_6)
- net RX3/15 is gone; now on net C2: J10.2 (Pin_2)
- net SDA/20 is gone; now on net SDA: J10.7 (Pin_7), J8.2 (Pin_2)
- net SDL is gone; now on net SCL: J11.2 (Pin_2), J13.8 (Pin_8)
- net TX0/1 is gone; now on net C0: J9.7 (Pin_7)
- net TX1/18 is gone; now on net ENC21: J10.5 (Pin_5)
- net TX2/16 is gone; now on net C3: J10.3 (Pin_3)
- net TX3/14 is gone; now on net C1: J10.1 (Pin_1)
- net AD0: no longer J13.4 (Pin_4)
- net GND: now also J13.4 (Pin_4)
- net VCC: now also SW2.2 (B), SW2.5 (B)
- net at con5.2 (Pin_2): now also SW2.3 (C), SW2.6 (C)
- net EDA: no longer names the net of J13.6 (Pin_6)
- net EDL: no longer names the net of J13.5 (Pin_5)
- net FYSINC: no longer names the net of J13.1 (Pin_1)
- net INT: no longer names the net of J13.3 (Pin_3)
- net NCS: no longer names the net of J13.2 (Pin_2)
- net SCL/21 renamed SCL
